Commit message: Add support files for ground cube pick-place demo

File: src/so101_gazebo/urdf/so101_gazebo.urdf (robot description, URDF)
Before this commit: robot so101_new_calib, 10 links, 9 joints
Joints:
- joint gripper_frame_joint: parent gripper_link -> wrist_link
- joint gripper_to_wrist_camera: origin xyz=0.055 0.0 0.020 rpy=0 1.5708 0 -> xyz=-0.0549 -0.0411 0.0154 rpy=1.6195 0 -1.5708; parent gripper_link -> wrist_link
